File: 02_Development/FlowMeter/Sensirion_connector_board/eagle/connector_board.brd (EAGLE design)
At the start: 19 x 20 mm, 13 parts

Commit message: added eagle files with changes
Parts:
- moved J7 5.08 mm to (-314.9, -287.8)
Routing:
- net GND: track 44.7 -> 54.8 mm
- net SDA1: track 41.1 -> 51.2 mm
- net 5V: track 31.9 -> 41.4 mm
- net SCL1: track 22.9 -> 32.3 mm
- net LY: track 23.4 -> 25.7 mm
Other:
- board size 19 x 20 mm -> 19 x 25.1 mm
