File: 02_Development/FlowMeter/RPi Board/PCB Design Files/raspberry_pi_v003.sch (EAGLE design)
At the start: 113 parts, among them J5 POWER_JACK, P1 SPL006-007, P2 SPL006-007, P3 SPL006-007, P4 SPL006-007, P5 SPL006-007, Q2 500mA/300V, U6 TCA9548APWR, U7 TCA9548APWR

Commit message: add new PCB v003 with updates (#135)
- added hard reset for sensirion using p-channel moseft
- added capacior per the updated cut sheet v1.6 for the 5V regulator
Parts:
- removed SP2: AL60P, buzzer:AL60P
- added C13: 33n, SparkFun-Capacitors:CAP-0805
- added Q1: 4.3A/20V/54mΩ, SparkFun-DiscreteSemi:MOSFET_PCH-IRLML2244
- added R47, R48: 10K, SparkFun-Resistors:0.3OHM-0805-1/8W-1%
Connections:
- new net SENS_POWER: J3.1, J7.1, J8.1, J9.1, Q1.D
- net 12V: no longer SP2.1
- net 3.3V: now also R48.1
- net 5V: now also C13.1
- net N$10: now also R48.2
- net N$11: now also C13.2
- net N$9: now also Q1.G, R47.1; no longer SP2.2
- net PI_5V_POWER: now also Q1.S, R47.2; no longer J3.1, J7.1, J8.1, J9.1
Other:
- note added: "Power For Flow Sensors"
- note added: "Q1 P-ch Mosfet MFR Part# AO3401A LCSC Part# C15127 Package SOT-23-3 https://datasheet.lcsc.com/szlcsc/Alpha-Omega-Semicon-AOS-AO3401A_C15127.pdf 1-gate, 2-source, 3-drain Q2 Transistor MFR Part# S8050 LCSC Part# C2146 Package SOT-23-3 NPN 500MA 25V https://datasheet.lcsc.com/szlcsc/Changjiang-Electronics-Tech-CJ-S8050_C2146.pdf 1-base, 2-emitter, 3-collector"
- note added: "version 003 - removed piezo buzzer - used transistor/P-ch mosfet for triggering sensirion power - added 33nF capacitor on the 5V power regulator based on rev1.6 of the data sheet"
- note removed: "Audio Alarm Generic Piezo w/6.5mm leads"
- note removed: "Q2 Transistor MFR Part# S8050 LCSC Part# C2146 Package SOT-23-3 NPN 500MA 25V https://datasheet.lcsc.com/szlcsc/Changjiang-Electronics-Tech-CJ-S8050_C2146.pdf 1-base, 2-emitter, 3-collector"
- moved on the sheet: Q2
