File: 02_Development/FlowMeter/RPi Board/PCB Design Files/raspberry_pi_v007.brd (EAGLE design)
At the start: 111.8 x 128.3 mm, 139 parts, among them J1 NP (277-2415-ND), J10 277-2419-ND, J11 POWER_JACK, J2 NP (277-2415-ND), J3 NP (277-2415-ND), J4 NP (277-2415-ND), J5 277-2419-ND, J6 277-2419-ND, J7 732-5315-ND, J8 277-2419-ND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

Commit message: Added power jumper, redid all manufacturing files & BOMs
Parts:
- added R59: 0R, SparkFun-Resistors:1206
- J11: value POWER_JACK -> CUI PJ-202A
- J7: value 732-5315-ND -> NP (732-5315-ND)
- J9: value 732-5315-ND -> Phoenix 1935776
Connections:
- net 5V: now also R59.2
- net PI_5V_POWER: now also R59.1
Routing:
- net PI_5V_POWER: track 198.3 -> 201.7 mm
- net 5V: track 73.1 -> 76.2 mm
Other:
- board text added: "Airflow and Pressure Sensor PI Hat Project Tetra Thomas Hudson et al. 11JAN2021 v0.00.007"
- board text removed: "Airflow and Pressure Sensor PI Hat Project Tetra Thomas Hudson et al. 06JAN2021 v0.00.007"
Changed lines of the file:
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@@
 <setting verticaltext="up"/>
 </settings>
-<grid distance="5" unitdist="mil" unit="mil" style="lines" multiple="1" display="no" altdistance="5" altunitdist="mil" altunit="mil"/>
+<grid distance="5" unitdist="mil" unit="mil" style="lines" multiple="1" display="yes" altdistance="5" altunitdist="mil" altunit="mil"/>
 <layers>
-<layer number="1" name="Top" color="4" fill="1" visible="yes" active="yes"/>
+<layer number="1" name="Top" color="4" fill="1" visible="no" active="yes"/>
 <layer number="2" name="Route2" color="1" fill="3" visible="no" active="no"/>
 <layer number="3" name="Route3" color="4" fill="3" visible="no" active="no"/>
@@
 <layer number="17" name="Pads" color="2" fill="1" visible="yes" active="yes"/>
 <layer number="18" name="Vias" color="2" fill="1" visible="yes" active="yes"/>
-<layer number="19" name="Unrouted" color="6" fill="1" visible="yes" active="yes"/>
+<layer number="19" name="Unrouted" color="6" fill="1" visible="no" active="yes"/>
 <layer number="20" name="Dimension" color="24" fill="1" visible="yes" active="yes"/>
 <layer number="21" name="tPlace" color="7" fill="1" visible="yes" active="yes"/>
-<layer number="22" name="bPlace" color="7" fill="1" visible="no" active="yes"/>
+<layer number="22" name="bPlace" color="7" fill="1" visible="yes" active="yes"/>
 <layer number="23" name="tOrigins" color="15" fill="1" visible="yes" active="yes"/>
-<layer number="24" name="bOrigins" color="15" fill="1" visible="no" active="yes"/>
+<layer number="24" name="bOrigins" color="15" fill="1" visible="yes" active="yes"/>
 <layer number="25" name="tNames" color="7" fill="1" visible="yes" active="yes"/>
 <layer number="26" name="bNames" color="7" fill="1" visible="no" active="yes"/>
 <layer number="27" name="tValues" color="7" fill="1" visible="no" active="yes"/>
 <layer number="28" name="bValues" color="7" fill="1" visible="no" active="yes"/>
-<layer number="29" name="tStop" color="7" fill="3" visible="no" active="yes"/>
+<layer number="29" name="tStop" color="7" fill="3" visible="yes" active="yes"/>
 <layer number="30" name="bStop" color="7" fill="6" visible="no" active="yes"/>
 <layer number="31" name="tCream" color="7" fill="4" visible="no" active="yes"/>
@@
 <layer number="37" name="tTest" color="7" fill="1" visible="no" active="yes"/>
 <layer number="38" name="bTest" color="7" fill="1" visible="no" active="yes"/>
-<layer number="39" name="tKeepout" color="4" fill="11" visible="yes" active="yes"/>
+<layer number="39" name="tKeepout" color="4" fill="11" visible="no" active="yes"/>
 <layer number="40" name="bKeepout" color="1" fill="11" visible="no" active="yes"/>
-<layer number="41" name="tRestrict" color="4" fill="10" visible="yes" active="yes"/>
+<layer number="41" name="tRestrict" color="4" fill="10" visible="no" active="yes"/>
 <layer number="42" name="bRestrict" color="1" fill="10" visible="no" active="yes"/>
 <layer number="43" name="vRestrict" color="2" fill="10" visible="no" active="yes"/>
@@
 <layer number="49" name="Reference" color="7" fill="1" visible="no" active="yes"/>
 <layer number="50" name="dxf" color="7" fill="1" visible="no" active="no"/>
-<layer number="51" name="tDocu" color="7" fill="1" visible="yes" active="yes"/>
+<layer number="51" name="tDocu" color="7" fill="1" visible="no" active="yes"/>
 <layer number="52" name="bDocu" color="7" fill="1" visible="no" active="yes"/>
 <layer number="53" name="tGND_GNDA" color="7" fill="9" visible="no" active="no"/>
@@
 </layers>
 <board>
-<fusionsync huburn="a.YnVzaW5lc3M6Z21haWw5OTQ5MjA" projecturn="a.YnVzaW5lc3M6Z21haWw5OTQ5MjAjMjAyMDA2MjkzMTE2MTgwMjY" f3durn="urn:adsk.wipprod:dm.lineage:n7ygfDT5Q_6xmTGKm0WD3Q" pcbguid="70598896-5c6f-486a-96a9-e9def747af8b" lastpulledtime="" lastsyncedchangeguid="" latestrevisionid="87264732-b09f-494d-9217-16bf7e0719ef" lastsyncedrevisionid="87264732-b09f-494d-9217-16bf7e0719ef" lastboardhashguid="54335742-8332-6d8e-25c5-1e5f82ced9bd" lastpushedtime="2021-01-06T20:09:17Z" linktopcb3d="true"/>
+<fusionsync huburn="a.YnVzaW5lc3M6Z21haWw5OTQ5MjA" projecturn="a.YnVzaW5lc3M6Z21haWw5OTQ5MjAjMjAyMDA2MjkzMTE2MTgwMjY" f3durn="urn:adsk.wipprod:dm.lineage:n7ygfDT5Q_6xmTGKm0WD3Q" pcbguid="" lastpulledtime="" lastsyncedchangeguid="" latestrevisionid="87264732-b09f-494d-9217-16bf7e0719ef" lastsyncedrevisionid="87264732-b09f-494d-9217-16bf7e0719ef" lastboardhashguid="54335742-8332-6d8e-25c5-1e5f82ced9bd" lastpushedtime="2021-01-06T20:09:17Z" linktopcb3d="true"/>
 <plain>
 <text x="-2.54" y="-47.498" size="1.4224" layer="21" font="vector" ratio="15" rot="R180">3V</text>
@@
 Project Tetra
 Thomas Hudson et al.
-06JAN2021
+11JAN2021
  v0.00.007</text>
 <text x="-29.7942" y="-23.1394" size="1.6764" layer="22" font="vector" ratio="15" rot="MR90" align="bottom-right">Sensirion Sensors #1-4</text>
@@
 <attribute name="VALUE" x="40.64" y="-10.795" size="1.016" layer="21" font="vector" ratio="15"/>
 </element>
-<element name="J11" library="SparkFun-Connectors" package="POWER_JACK_PTH" value="POWER_JACK" x="38.1" y="-59.69" smashed="yes">
+<element name="J11" library="SparkFun-Connectors" package="POWER_JACK_PTH" value="CUI PJ-202A" x="38.1" y="-59.69" smashed="yes">
 <attribute name="PROD_ID" value="CONN-08197" x="38.1" y="-59.69" size="1.778" layer="27" display="off"/>
 </element>
@@
 <attribute name="VALUE" x="5.588" y="-36.068" size="1.016" layer="21" font="vector" ratio="15" align="top-center"/>
 </element>
-<element name="J7" library="SparkFun-Connectors" package="1X02" value="732-5315-ND" x="2.54" y="-31.75" smashed="yes">
+<element name="J7" library="SparkFun-Connectors" package="1X02" value="NP (732-5315-ND)" x="2.54" y="-31.75" smashed="yes">
 <attribute name="VALUE" x="1.27" y="-33.782" size="0.6096" layer="27" font="vector" ratio="20"/>
 </element>
-<element name="J9" library="SparkFun-Connectors" package="SCREWTERMINAL-5MM-2" value="732-5315-ND" x="-15.113" y="-52.07" smashed="yes">
+<element name="J9" library="SparkFun-Connectors" package="SCREWTERMINAL-5MM-2" value="Phoenix 1935776" x="-15.113" y="-52.07" smashed="yes">
 <attribute name="SF_SKU" value="PRT-08432" x="-15.113" y="-52.07" size="1.016" layer="27" ratio="15" display="off"/>
 <attribute name="VALUE" x="-16.383" y="-50.8" size="0.6096" layer="27" font="vector" ratio="20"/>
@@
 <element name="FD3" library="Fiducial" package="FID_040" value="FID_40MIL" x="-14.097" y="55.118" smashed="yes">
 <attribute name="BOM" value="" x="-14.097" y="55.118" size="1.778" layer="27" display="off"/>
+</element>
+<element name="R59" library="SparkFun-Resistors" library_urn="urn:adsk.eagle:library:532" package="1206" package3d_urn="urn:adsk.eagle:package:39654/1" value="0R" x="3.429" y="-28.575" smashed="yes">
+<attribute name="NAME" x="0.889" y="-28.575" size="0.6096" layer="25" font="vector" ratio="20" rot="R90" align="bottom-center"/>
+<attribute name="PROD_ID" value=" " x="3.429" y="-28.575" size="1.778" layer="27" display="off"/>
+<attribute name="VALUE" x="3.429" y="-29.464" size="0.6096" layer="27" font="vector" ratio="20" align="top-center"/>
 </element>
 </elements>
@@
 <wire x1="4.953" y1="-22.606" x2="4.953" y2="-31.623" width="1.27" layer="1"/>
 <wire x1="4.953" y1="-31.623" x2="5.08" y2="-31.75" width="1.27" layer="1"/>
+<contactref element="R59" pad="2"/>
+<wire x1="4.829" y1="-28.575" x2="4.953" y2="-28.699" width="0.1524" layer="1"/>
+<wire x1="4.953" y1="-28.699" x2="4.953" y2="-31.623" width="0.1524" layer="1"/>
 </signal>
 <signal name="A0_PC">
@@
 <wire x1="39.624" y1="-6.096" x2="39.624" y2="-4.826" width="0.6096" layer="1"/>
 <wire x1="0" y1="-4.826" x2="0.762" y2="-4.064" width="0.6096" layer="1"/>
+<contactref element="R59" pad="1"/>
+<wire x1="2.029" y1="-28.575" x2="2.54" y2="-29.086" width="0.1524" layer="1"/>
+<wire x1="2.54" y1="-29.086" x2="2.54" y2="-31.75" width="0.1524" layer="1"/>
 </signal>
 <signal name="5VREG-SW">
